Commit message: Align robot URDF with Gazebo, improve robot_description meshes, tune RL stack.
Fix visual mesh orientation and lidar joint in URDF; resolve file:// and
package:// mesh URIs in emit_robot_description; add lidar clearance parameter;
refactor rl_train and update Gazebo bridge and launch scripts.

Co-authored-by: Cursor <cursoragent@cursor.com>

File: course_robot/course_robot.urdf (robot description, URDF)
Before this commit: robot course_robot, 2 links, 1 joints
Joints:
- joint lidar_joint: origin xyz=0.13 0 0.17 rpy=0 0 0 -> xyz=-0.05 0 0.15 rpy=0 0 0
